Commit message: pendulum urdf

File: pendulum.urdf (robot description, URDF)
Before this commit: robot pendulum, 2 links, 1 joints
Links:
- added link axe, mass 0; visual cylinder length=0.5 radius=0.005
- added link eef, mass 1; visual sphere radius=0.03
- link base: geometry visual sphere radius=0.05
Joints:
- added joint j1: type revolute, parent base, child axe, origin xyz=0 0 0 rpy=0.5 0 0, axis 1 0 0, limit effort=0 velocity=0
- added joint j2: type fixed, parent axe, child eef, origin xyz=0 0 -0.5 rpy=0 0 0
- joint world_to_base: origin xyz=0 0 1 rpy=0 0 0 -> xyz=0 0 2 rpy=0 0 0

Commit message: freely moving pendulum

File: pendulum.urdf (robot description, URDF)
Before this commit: robot pendulum, 4 links, 3 joints
Joints:
- joint j1: origin xyz=0 0 0 rpy=0.5 0 0 -> xyz=0 0 0 rpy=0 0 0
